Commit message: Update gp12_macro.xacro

File: motoman_gp12_support/urdf/gp12_macro.xacro (robot description, xacro)
@@ -5,4 +5,9 @@
     <!-- link list -->
     <link name="${prefix}base_link">
+        <inertial>
+          <mass value="21.63"/>
+          <origin xyz="-0.05823927 0.000903 0.08108367"/>
+          <inertia ixx="0.0001828580709370491" ixy="2.267080402506378e-06" ixz="5.437316910269656e-07" iyx="2.267080402506378e-06" iyy="0.0003096397167638798" iyz="-2.118890055125151e-06" izx="5.437316910269656e-07" izy="-2.118890055125151e-06" izz="0.0004048893615748322"/>
+        </inertial>
         <visual>
             <geometry>
@@ -18,4 +23,9 @@
     </link>
     <link name="${prefix}link_1_s">
+        <inertial>
+          <mass value="39.88"/>
+          <origin xyz="0.03208235 0.0025694 -0.13315049"/>
+          <inertia ixx="0.0006540366623769821" ixy="-2.3218347207311178e-05" ixz="-0.00015971907483118441" iyx="-2.3218347207311178e-05" iyy="0.0007288556603654311" iyz="-1.1799196009268088e-05" izx="-0.00015971907483118441" izy="-1.1799196009268088e-05" izz="0.0007274290536849057"/>
+        </inertial>
         <visual>
             <geometry>
@@ -31,4 +41,9 @@
     </link>
     <link name="${prefix}link_2_l">
+        <inertial>
+          <mass value="15.97"/>
+          <origin xyz="-0.01081779 -0.10730189 0.28700609"/>
+          <inertia ixx="0.0005892591420666659" ixy="-4.833499831620306e-06" ixz="-4.3155628473392336e-06" iyx="-4.833499831620306e-06" iyy="0.0005996513130448696" iyz="1.0912822055333276e-05" izx="-4.3155628473392336e-06" izy="1.0912822055333276e-05" izz="5.132964626776372e-05"/>
+        </inertial>
         <visual>
             <geometry>
@@ -44,4 +59,9 @@
     </link>
     <link name="${prefix}link_3_u">
+        <inertial>
+          <mass value="21.26"/>
+          <origin xyz="0.09599858 -0.02713391 0.10938789"/>
+          <inertia ixx="0.0002739752053986467" ixy="1.5549400208507755e-05" ixz="-8.915090110642345e-05" iyx="1.5549400208507755e-05" iyy="0.0002841703943472267" iyz="2.7348827905335803e-05" izx="-8.915090110642345e-05" izy="2.7348827905335803e-05" izz="0.0002453524128147622"/>
+        </inertial>
         <visual>
             <geometry>
@@ -57,4 +77,9 @@
     </link>
     <link name="${prefix}link_4_r">
+        <inertial>
+          <mass value="10.62"/>
+          <origin xyz="-0.17042382 0.00328433 0.00535304"/>
+          <inertia ixx="3.800959525449092e-05" ixy="1.0709973017466907e-06" ixz="3.1285422077393913e-06" iyx="1.0709973017466907e-06" iyy="0.00015385961557079752" iyz="-5.011203255667548e-07" izx="3.1285422077393913e-06" izy="-5.011203255667548e-07" izz="0.0001634833979445244"/>
+        </inertial>
         <visual>
             <geometry>
@@ -70,4 +95,9 @@
     </link>
     <link name="${prefix}link_5_b">
+        <inertial>
+          <mass value="2.04"/>
+          <origin xyz="0.02902053 -0.00034857 -0.00119948"/>
+          <inertia ixx="4.114182064247773e-06" ixy="3.04837248361879e-08" ixz="-1.3212217694437561e-07" iyx="3.04837248361879e-08" iyy="4.822066900949523e-06" iyz="7.993041826670504e-08" izx="-1.3212217694437561e-07" izy="7.993041826670504e-08" izz="5.173348542964499e-06"/>
+        </inertial>
         <visual>
             <geometry>
@@ -83,4 +113,9 @@
     </link>
     <link name="${prefix}link_6_t">
+        <inertial>
+          <mass value="0.0197"/>
+          <origin xyz="9.69962575e-02 1.04417964e-11 -3.09900584e-11"/>
+          <inertia ixx="8.644578899728899e-09" ixy="3.134772128194266e-15" ixz="1.3008517244263161e-17" iyx="3.134772128194266e-15" iyy="4.376299175251843e-09" iyz="3.8745545703522195e-18" izx="1.3008517244263161e-17" izy="3.8745545703522195e-18" izz="4.376295928866491e-09"/>
+        </inertial>
         <visual>
             <geometry>
